File: bio-chemistry-analyzer/biochem_M_V2.sch (EAGLE design)
At the start: 37 parts, among them J1 61201021621, J2 USB1135-15-9-L-B_REVA1, Q4-T IRFZ44N, Q4-T4 IRFZ44N, Q4-T5 IRFZ44N, Q4-T6 IRFZ44N

Commit message: PCB Changes
Parts:
- removed 10KR1, 10KR4: (no value), rcl:R-US_0204/7
- removed PELT1, PELT2: B4B-XH-2PIN2PIN, B4B-XH-A_LF__SN_:B4B-XH-2PIN2PIN
- removed Q4-T5, Q4-T6: IRFZ44N, IRFZ44N:IRFZ44N
- added U$2: MDD3A, MDD3A:MDD3A
Connections:
- removed net N$3: JP1.4, SV1.7
- removed net N$6: JP1.5, SV1.9
- removed net PELT1: 10KR4.2, JP2.3, Q4-T5.G, SV1.36
- removed net PELT2: 10KR1.2, JP1.6, Q4-T6.G, SV1.11
- removed net PELTIER1: PELT1.1, Q4-T5.D
- removed net PELTIER2: PELT2.1, Q4-T6.D
- new net PELT1A: JP2.3, SV1.36, U$2.M1AIN
- new net PELT1B: JP1.4, SV1.7, U$2.M1BIN
- new net PELT2A: JP1.6, SV1.11, U$2.M2AIN
- new net PELT2B: JP1.5, SV1.9, U$2.M2BIN
- net 5V: now also U$2.5V; no longer PELT1.2, PELT2.2
- net GND: now also U$2.GND; no longer 10KR1.1, 10KR4.1, Q4-T5.S, Q4-T6.S

Commit message: requirements
Parts:
- added U$3: QRBIOS, Logo:QRBIOS
Changed lines of the file:
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@@
 <part name="J2" library="USB1135-15-9-L-B_REVA1" deviceset="USB1135-15-9-L-B_REVA1" device=""/>
 <part name="U$2" library="MDD3A" deviceset="MDD3A" device=""/>
+<part name="U$3" library="Logo" deviceset="QRBIOS" device=""/>
 </parts>
 <sheets>
@@
 </instance>
 <instance part="U$2" gate="G$1" x="375.92" y="33.02" smashed="yes"/>
+<instance part="U$3" gate="G$1" x="228.6" y="182.88" smashed="yes"/>
 </instances>
 <busses>
